Commit message: implemented contact estimation with momentum residual

File: 01-model_based_baseline/4pbot_fixed.urdf (robot description, URDF)
Before this commit: robot 4pbot, 5 links, 4 joints
Links:
- link link2: geometry collision box size=0.04 0.10 0.9; visual box size=0.04 0.10 1.0
- link link3: geometry collision box size=0.04 0.10 0.9; visual box size=0.04 0.10 1.0

Commit message: improved the controller and the plotting functions

File: 01-model_based_baseline/4pbot_fixed.urdf (robot description, URDF)
Before this commit: robot 4pbot, 5 links, 4 joints
Links:
- link link4: geometry collision box size=0.04 0.10 0.9; visual box size=0.04 0.10 1.0
